File: Hardware/Serial Controlled Motor Driver.brd (EAGLE design)
At the start: 20.3 x 38.1 mm, 49 parts, among them J1 DNP, J2 DNP, J3 DNP, J4 DNP, J5 DNP, J6 DNP, J7 DNP, J8 CORTEX_DEBUGPTH, U1 CY8C4245LQI-483, U2 DRV8835

Commit message: Fixed proto errors and started final API for arduino
Connections:
- net CONFIG_IN: now also J4.4, U1.11; no longer J4.5, R3.1, U1.10
- net CONFIG_OUT: now also J4.5, R3.1, U1.10; no longer J4.4, U1.11
Routing:
- net CONFIG_OUT: track 11.2 -> 12.3 mm
- net CONFIG_IN: track 12.3 -> 11.2 mm
Changed lines of the file:
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@@
 <layer number="15" name="Route15" color="4" fill="6" visible="no" active="no"/>
 <layer number="16" name="Bottom" color="1" fill="1" visible="yes" active="yes"/>
-<layer number="17" name="Pads" color="2" fill="1" visible="no" active="yes"/>
-<layer number="18" name="Vias" color="2" fill="1" visible="no" active="yes"/>
-<layer number="19" name="Unrouted" color="6" fill="1" visible="no" active="yes"/>
-<layer number="20" name="Dimension" color="15" fill="1" visible="no" active="yes"/>
-<layer number="21" name="tPlace" color="16" fill="1" visible="no" active="yes"/>
-<layer number="22" name="bPlace" color="14" fill="1" visible="no" active="yes"/>
-<layer number="23" name="tOrigins" color="15" fill="1" visible="no" active="yes"/>
-<layer number="24" name="bOrigins" color="15" fill="1" visible="no" active="yes"/>
+<layer number="17" name="Pads" color="2" fill="1" visible="yes" active="yes"/>
+<layer number="18" name="Vias" color="2" fill="1" visible="yes" active="yes"/>
+<layer number="19" name="Unrouted" color="6" fill="1" visible="yes" active="yes"/>
+<layer number="20" name="Dimension" color="15" fill="1" visible="yes" active="yes"/>
+<layer number="21" name="tPlace" color="16" fill="1" visible="yes" active="yes"/>
+<layer number="22" name="bPlace" color="14" fill="1" visible="yes" active="yes"/>
+<layer number="23" name="tOrigins" color="15" fill="1" visible="yes" active="yes"/>
+<layer number="24" name="bOrigins" color="15" fill="1" visible="yes" active="yes"/>
 <layer number="25" name="tNames" color="7" fill="1" visible="no" active="yes"/>
 <layer number="26" name="bNames" color="7" fill="1" visible="no" active="yes"/>
 <layer number="27" name="tValues" color="7" fill="1" visible="no" active="yes"/>
 <layer number="28" name="bValues" color="7" fill="1" visible="no" active="yes"/>
-<layer number="29" name="tStop" color="7" fill="3" visible="yes" active="yes"/>
-<layer number="30" name="bStop" color="7" fill="6" visible="yes" active="yes"/>
+<layer number="29" name="tStop" color="7" fill="3" visible="no" active="yes"/>
+<layer number="30" name="bStop" color="7" fill="6" visible="no" active="yes"/>
 <layer number="31" name="tCream" color="7" fill="4" visible="no" active="yes"/>
 <layer number="32" name="bCream" color="7" fill="5" visible="no" active="yes"/>
@@
 <layer number="43" name="vRestrict" color="2" fill="10" visible="no" active="yes"/>
 <layer number="44" name="Drills" color="7" fill="1" visible="no" active="yes"/>
-<layer number="45" name="Holes" color="7" fill="1" visible="no" active="yes"/>
+<layer number="45" name="Holes" color="7" fill="1" visible="yes" active="yes"/>
 <layer number="46" name="Milling" color="3" fill="1" visible="no" active="yes"/>
 <layer number="47" name="Measures" color="7" fill="1" visible="no" active="yes"/>
@@
 <layer number="49" name="Reference" color="7" fill="1" visible="no" active="yes"/>
 <layer number="50" name="dxf" color="7" fill="1" visible="no" active="no"/>
-<layer number="51" name="tDocu" color="6" fill="1" visible="no" active="yes"/>
+<layer number="51" name="tDocu" color="6" fill="1" visible="yes" active="yes"/>
 <layer number="52" name="bDocu" color="7" fill="1" visible="no" active="yes"/>
 <layer number="53" name="tGND_GNDA" color="7" fill="9" visible="no" active="no"/>
@@
 <wire x1="8.64" y1="12.719875" x2="8.64" y2="14.78" width="0.254" layer="1"/>
 </signal>
-<signal name="CONFIG_OUT">
+<signal name="CONFIG_IN">
 <contactref element="J4" pad="4"/>
 <contactref element="U1" pad="11"/>
@@
 <wire x1="3.413125" y1="20.875625" x2="2.57175" y2="20.03425" width="0.254" layer="1"/>
 </signal>
-<signal name="CONFIG_IN">
+<signal name="CONFIG_OUT">
 <contactref element="J4" pad="5"/>
 <contactref element="R3" pad="1"/>

Commit message: Added Byron's review suggestions
Other:
- board text added: "MAX 11V"
- board text added: "v20"
- board text removed: "+3- 11V"
- board text removed: "v16"
